Commit message: Update macro.xacro
Parametrizing the collision name like visuals

File: my_first_robot/urdf/macro.xacro (robot description, xacro)
@@ -15,5 +15,5 @@
               <inertia ixx="0.000526666666667" ixy="0" ixz="0" iyy="0.000526666666667" iyz="0" izz="0.001"/>
             </inertial>
-            <collision name="link_right_wheel_collision">
+            <collision name="${name}_collision">
               <origin rpy="0 1.5707 1.5707" xyz="0 0 0"/>
               <geometry>
